File: esc/esc.kicad_pcb (KiCad board)
At the start: 2 copper layers, 52.1 x 20.3 mm, 33 parts, among them J1 USB_C_Receptacle_USB2.0, U1 XC6206P332MR, U2 STM32F103CBT6, Y1 8M, Y2 NM (32.768k)

Commit message: Hmmmm
Parts:
- removed C10, C11, C8, C9: 20pF, Capacitor_SMD:C_0402_1005Metric
- removed C3: 10uF, Capacitor_SMD:C_0603_1608Metric
- removed C4, C5, C6, C7: 100nF, Capacitor_SMD:C_0402_1005Metric
- removed D2: YEL, LED_SMD:LED_0603_1608Metric
- removed D3: BLUE, LED_SMD:LED_0603_1608Metric
- removed J2: ~, Connector_PinHeader_2.54mm:PinHeader_2x03_P2.54mm_Horizontal
- removed R1, R5: NM, Resistor_SMD:R_0402_1005Metric
- removed R2, R3: 22R, Resistor_SMD:R_0402_1005Metric
- removed R4: 1.5k, Resistor_SMD:R_0402_1005Metric
- removed R6, R7: 5.1k, Resistor_SMD:R_0402_1005Metric
- removed R8, R9: 470, Resistor_SMD:R_0402_1005Metric
- removed SW1, SW2: ~, Button_Switch_SMD:SW_SPST_TL3342
- removed U2: STM32F103CBT6, Package_QFP:LQFP-48_7x7mm_P0.5mm
- removed Y1: 8M, Crystal:Crystal_SMD_Abracon_ABM3-2Pin_5.0x3.2mm
- removed Y2: NM (32.768k), Crystal:Crystal_SMD_EuroQuartz_EQ161-2Pin_3.2x1.5mm
- added Q1: NCEP60T12AK, Package_TO_SOT_SMD:TO-252-2, F.Cu at (195.6, 128.5)
- added Q2: NCEP60T12AK, Package_TO_SOT_SMD:TO-252-2, B.Cu at (195.6, 128.3)
- C1: value 10uF -> C
- C2: value 100nF -> C; footprint Capacitor_SMD:C_0402_1005Metric -> Capacitor_SMD:C_0603_1608Metric
- D1: footprint Diode_SMD:D_SOD-123 -> Diode_SMD:D_SOD-323
- J1: value USB_C_Receptacle_USB2.0 -> ~; footprint Connector_USB:USB_C_Receptacle_HRO_TYPE-C-31-M-12 -> TestPoint:TestPoint_Plated_Hole_D3.0mm; moved to F.Cu
- U1: value XC6206P332MR -> IR2101; footprint Package_TO_SOT_SMD:SOT-23 -> Package_SO:SOIC-8_3.9x4.9mm_P1.27mm
- moved J1 37.9 mm to (195.6, 139.1), turned to 0 degrees
- moved D1 33.3 mm to (167.6, 118.7), turned to 180 degrees
- moved C1 33.0 mm to (165.1, 118.7)
- moved U1 30.9 mm to (167.6, 123.2), turned to 0 degrees
- moved C2 18.5 mm to (170.2, 118.7), turned to 90 degrees
Connections:
- C1 pad 1: +5V -> +3V3
- C2 pad 1: RST -> +12V
- D1 pad 1: +5V -> +12V
- D1 pad 2: VBUS -> +3V3
- U1 pad 1: GND -> +3V3
- U1 pad 2: +3V3 -> CAH
- U1 pad 3: +5V -> CAL
Routing:
- net +3V3: track 141.7 -> 0.00 mm, vias 3 -> 0
- net RST: track 47.6 -> 0.00 mm, vias 4 -> 0
- net C13: track 41.0 -> 0.00 mm, vias 2 -> 0
- net C14: track 34.7 -> 0.00 mm
- net SWDIO: track 34.7 -> 0.00 mm, vias 1 -> 0
- net B3: track 32.6 -> 0.00 mm, vias 1 -> 0
- net A12: track 30.1 -> 0.00 mm, vias 2 -> 0
- net SWCLK: track 29.7 -> 0.00 mm, vias 1 -> 0
- net BO0: track 27.0 -> 0.00 mm, vias 2 -> 0
- net C15: track 26.8 -> 0.00 mm
- net A11: track 26.0 -> 0.00 mm, vias 2 -> 0
- net B12: track 19.4 -> 0.00 mm
- net B9: track 17.3 -> 0.00 mm
- net B13: track 17.1 -> 0.00 mm
- net A0: track 16.2 -> 0.00 mm
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- removed copper zone on B.Cu, net VBUS
- removed copper zone on F.Cu, net VBUS
Other:
- board size 52.1 x 20.3 mm -> 52.1 x 52.1 mm

Commit message: Hmmm
Parts:
- added J2: ~, TestPoint:TestPoint_Plated_Hole_D3.0mm, F.Cu at (169.2, 122.4)
- added J5: ~, TestPoint:TestPoint_Plated_Hole_D3.0mm, F.Cu at (169.2, 128.5)
- added U2: TPS5430DDA, Package_SO:TI_SO-PowerPAD-8_ThermalVias, F.Cu at (161.9, 122.7)
- Q1: moved to B.Cu
- Q2: moved to F.Cu
- moved D1 28.2 mm to (195.6, 115.2)
- moved U1 28.2 mm to (195.6, 119.6)
- moved C1 28.2 mm to (193.0, 115.2)
- moved C2 28.2 mm to (198.1, 115.2)
- moved Q2 3.57 mm to (192.0, 128.5)
- moved Q1 3.56 mm to (192.0, 128.5)
Connections:
- C2 pad 1: +12V -> VDC
- D1 pad 1: +12V -> VDC
- U1 pad 8: +12V -> VDC
Other:
- board text removed: "CLK/IO"
- board text removed: "GND/SWO"
- board text removed: "RST/3V3"
