File: pcb/gp.kicad_sch (KiCad schematic)
At the start: 31 parts, among them J1 USB-C, SW1 TS-1088R-02526, SW2 TS-1088R-02526, U1 XC6206P332MR, U2 STM32F103CBT6, U3 W25Q32JVSS, Y1 16Mhz

Commit message: Hmmm
Parts:
- U3: value W25Q32JVSS -> W25Q128JVSIQ; footprint Package_SO:SOIC-8_5.23x5.23mm_P1.27mm -> Package_SO:SOIC-8_5.3x5.3mm_P1.27mm; LCSC (none) -> C97521
Changed lines of the file:
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@@
 			)
 		)
-		(property "Value" "W25Q32JVSS"
+		(property "Value" "W25Q128JVSIQ"
 			(at 154.94 149.86 0)
 			(effects
@@
 			)
 		)
-		(property "Footprint" "Package_SO:SOIC-8_5.23x5.23mm_P1.27mm"
+		(property "Footprint" "Package_SO:SOIC-8_5.3x5.3mm_P1.27mm"
 			(at 146.05 158.75 0)
 			(effects
@@
 			)
 		)
+		(property "LCSC" "C97521"
+			(at 146.05 158.75 0)
+			(effects
+				(font
+					(size 1.27 1.27)
+				)
+				(hide yes)
+			)
+		)

Commit message: Minor rev. d changes
Connections:
- net A15: no longer U3.1 (~{CS})
- net A4: now also U3.1 (~{CS})
- net A5: now also U3.6 (CLK)
- net A6: now also U3.2 (DO(IO1))
- net A7: now also U3.5 (DI(IO0))
- net B3: no longer U3.6 (CLK)
- net B4: no longer U3.2 (DO(IO1))
- net B5: no longer U3.5 (DI(IO0))
- net BO0: now also U2.22 (PB11)
- no-connect marks 6 -> 5
Changed lines of the file:
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@@
 	(text "Reset & Boot Mode"
 		(exclude_from_sim no)
-		(at 13.97 127 0)
+		(at 13.97 128.27 0)
 		(effects
 			(font
@@
 	(text "Programming Header"
 		(exclude_from_sim no)
-		(at 179.07 127 0)
+		(at 179.07 128.27 0)
 		(effects
 			(font
@@
 	(text "LEDs"
 		(exclude_from_sim no)
-		(at 72.39 127 0)
+		(at 72.39 128.27 0)
 		(effects
 			(font
@@
 	(text "EEPROM"
 		(exclude_from_sim no)
-		(at 123.19 127 0)
+		(at 114.3 128.27 0)
 		(effects
 			(font
@@
 	)
 	(no_connect
-		(at 170.18 90.17)
-	)
-	(no_connect
 		(at 158.75 161.29)
 	)
@@
 	(wire
 		(pts
-			(xy 167.64 34.29) (xy 170.18 34.29)
+			(xy 161.29 34.29) (xy 170.18 34.29)
+		)
+		(stroke
+			(width 0)
+			(type default)
+		)
+	)
+	(wire
+		(pts
+			(xy 161.29 90.17) (xy 170.18 90.17)
 		)
 		(stroke
@@
 	(wire
 		(pts
-			(xy 167.64 39.37) (xy 170.18 39.37)
+			(xy 161.29 39.37) (xy 170.18 39.37)
 		)
 		(stroke
@@
 		)
 	)
-	(global_label "B5"
-		(shape input)
-		(at 161.29 153.67 0)
-		(fields_autoplaced yes)
-		(effects
-			(font
-				(size 1.27 1.27)
-			)
-			(justify left)
-		)
-		(property "Intersheetrefs" "${INTERSHEET_REFS}"
-			(at -53.34 11.43 0)
-			(effects
-				(font
-					(size 1.27 1.27)
-				)
-				(hide yes)
-			)
-		)
-	)
 	(global_label "SWCLK"
 		(shape input)
@@
 		)
 	)
-	(global_label "A15"
+	(global_label "A5"
 		(shape input)
-		(at 130.81 156.21 180)
+		(at 130.81 161.29 180)
 		(fields_autoplaced yes)
 		(effects
@@
 		)
 		(property "Intersheetrefs" "${INTERSHEET_REFS}"
-			(at -53.34 11.43 0)
+			(at 126.1809 161.29 0)
 			(effects
 				(font
 					(size 1.27 1.27)
 				)
+				(justify right)
 				(hide yes)
 			)
@@
 		)
 	)
+	(global_label "A6"
+		(shape input)
+		(at 161.29 156.21 0)
+		(fields_autoplaced yes)
+		(effects
+			(font
+				(size 1.27 1.27)
+			)
+			(justify left)
+		)
+		(property "Intersheetrefs" "${INTERSHEET_REFS}"
+			(at -52.07 73.66 0)
+			(effects
+				(font
+					(size 1.27 1.27)
+				)
+				(hide yes)
+			)
+		)
+	)
 	(global_label "A7"
 		(shape input)
@@
 		)
 	)
-	(global_label "B3"
-		(shape input)
-		(at 130.81 161.29 180)
-		(fields_autoplaced yes)
-		(effects
-			(font
-				(size 1.27 1.27)
-			)
-			(justify right)
-		)
-		(property "Intersheetrefs" "${INTERSHEET_REFS}"
-			(at -53.34 11.43 0)
-			(effects
-				(font
-					(size 1.27 1.27)
-				)
-				(hide yes)
-			)
-		)
-	)
 	(global_label "A11"
 		(shape input)
@@
 	(global_label "BO0"
 		(shape input)
-		(at 167.64 39.37 180)
+		(at 161.29 39.37 180)
 		(fields_autoplaced yes)
 		(effects
@@
 		)
 		(property "Intersheetrefs" "${INTERSHEET_REFS}"
-			(at -7.62 -5.08 0)
+			(at -13.97 -5.08 0)
 			(effects
 				(font
@@
 		)
 	)
+	(global_label "A4"
+		(shape input)
+		(at 130.81 156.21 180)
+		(fields_autoplaced yes)
+		(effects
+			(font
+				(size 1.27 1.27)
+			)
+			(justify right)
+		)
+		(property "Intersheetrefs" "${INTERSHEET_REFS}"
+			(at 126.1809 156.21 0)
+			(effects
+				(font
+					(size 1.27 1.27)
+				)
+				(justify right)
+				(hide yes)
+			)
+		)
+	)
 	(global_label "B13"
 		(shape input)
@@
 	(global_label "RST"
 		(shape input)
-		(at 167.64 34.29 180)
+		(at 161.29 34.29 180)
 		(fields_autoplaced yes)
 		(effects
@@
 		)
 		(property "Intersheetrefs" "${INTERSHEET_REFS}"
-			(at -7.62 -5.08 0)
+			(at -13.97 -5.08 0)
 			(effects
 				(font
@@
 		)
 	)
+	(global_label "BO0"
+		(shape input)
+		(at 161.29 90.17 180)
+		(fields_autoplaced yes)
+		(effects
+			(font
+				(size 1.27 1.27)
+			)
+			(justify right)
+		)
+		(property "Intersheetrefs" "${INTERSHEET_REFS}"
+			(at -13.97 45.72 0)
+			(effects
+				(font
+					(size 1.27 1.27)
+				)
+				(hide yes)
+			)
+		)
+	)
 	(global_label "B14"
 		(shape input)
@@
 		)
 	)
-	(global_label "BO0"
+	(global_label "A7"
 		(shape input)
-		(at 57.15 158.75 0)
+		(at 161.29 153.67 0)
 		(fields_autoplaced yes)
 		(effects
@@
 		)
 		(property "Intersheetrefs" "${INTERSHEET_REFS}"
-			(at 63.291 158.75 0)
+			(at -52.07 68.58 0)
 			(effects
 				(font
 					(size 1.27 1.27)
 				)
-				(justify left)
 				(hide yes)
 			)
 		)
 	)
-	(global_label "B15"
+	(global_label "BO0"
 		(shape input)
-		(at 161.29 100.33 180)
+		(at 57.15 158.75 0)
 		(fields_autoplaced yes)
 		(effects
@@
 				(size 1.27 1.27)
 			)
-			(justify right)
+			(justify left)
 		)
 		(property "Intersheetrefs" "${INTERSHEET_REFS}"
-			(at -7.62 -5.08 0)
+			(at 63.291 158.75 0)
 			(effects
 				(font
 					(size 1.27 1.27)
 				)
+				(justify left)
 				(hide yes)
 			)
 		)
 	)
-	(global_label "B4"
+	(global_label "B15"
 		(shape input)
-		(at 161.29 156.21 0)
+		(at 161.29 100.33 180)
 		(fields_autoplaced yes)
 		(effects
@@
 				(size 1.27 1.27)
 			)
-			(justify left)
+			(justify right)
 		)
 		(property "Intersheetrefs" "${INTERSHEET_REFS}"
-			(at -53.34 11.43 0)
+			(at -7.62 -5.08 0)
 			(effects
 				(font

Commit message: More fine tuning of PCB
Parts:
- D2: value GRE -> WHI; LCSC C72043 -> C2290
- D3: LCSC C72041 -> C2288
Changed lines of the file:
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@@
 			)
 		)
-		(property "Value" "GRE"
+		(property "Value" "WHI"
 			(at 81.28 157.48 90)
 			(effects
@@
 			)
 		)
-		(property "LCSC" "C72043"
+		(property "LCSC" "C2290"
 			(at 77.47 154.94 90)
 			(effects
@@
 			)
 		)
-		(property "LCSC" "C72041"
+		(property "LCSC" "C2288"
 			(at 86.36 154.94 90)
 			(effects

Commit message: Tweaks
Parts:
- added C4, C9: 100nF, Capacitor_SMD:C_0402_1005Metric, symbol Device:C
- renumbered C8 to C10, C9 to C11, C4 to C5, C5 to C6, C6 to C7, C7 to C8, R5 to R2, R2 to R3, R3 to R4, R4 to R5, R8 to R6, R6 to R7, R9 to R8, R7 to R9, U3 to U2, U2 to U3
Connections:
- net +3V3: now also C9.1
- net BO0: now also C4.1
- net GND: now also C4.2, C9.2
Other:
- note added: "MCU"
- note removed: "Processor"
- moved on the sheet: C1, C10, C11, C2, C3, C5, C6, C7, C8, D1, D2, D3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
