File: pcb/gp.kicad_pcb (KiCad board)
At the start: 2 copper layers, 52.1 x 20.3 mm, 31 parts, among them J1 USB-C, SW1 TS-1088R-02526, SW2 TS-1088R-02526, U1 XC6206P332MR, U2 STM32F103CBT6, U3 W25Q128JVSIQ, Y1 16Mhz

Commit message: Hmmmm
Routing:
- net B3: track 35.2 -> 34.6 mm
- net GND: vias 18 -> 21
Changed lines of the file:
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@@
+	)
+	(via
+		(at 187.96 103.505)
+		(size 0.7)
+		(drill 0.35)
+		(layers "F.Cu" "B.Cu")
+		(free yes)
+		(net 1)
 	)
 	(via
@@
 	)
 	(via
+		(at 165.735 97.155)
+		(size 0.7)
+		(drill 0.35)
+		(layers "F.Cu" "B.Cu")
+		(free yes)
+		(net 1)
+	)
+	(via
 		(at 171.45 106.045)
 		(size 0.7)
@@
 	)
 	(via
+		(at 188.976 104.648)
+		(size 0.7)
+		(drill 0.35)
+		(layers "F.Cu" "B.Cu")
+		(net 1)
+	)
+	(via
 		(at 174.625 100.33)
 		(size 0.7)
@@
 	)
 	(via
-		(at 189.23 105.41)
+		(at 188.976 105.41)
 		(size 0.7)
 		(drill 0.35)
@@
 	)
 	(via
-		(at 189.23 104.14)
+		(at 187.96 102.616)
 		(size 0.7)
 		(drill 0.35)
@@
 	)
 	(segment
-		(start 162.135 98.425)
-		(end 165.1 98.425)
-		(width 0.2286)
-		(layer "F.Cu")
-		(net 13)
-	)
-	(segment
 		(start 174.922 96.882126)
 		(end 174.922 95.588)
@@
 	)
 	(segment
-		(start 165.1 98.425)
-		(end 165.735 97.79)
+		(start 162.135 98.425)
+		(end 165.735 98.425)
 		(width 0.2286)
 		(layer "F.Cu")
@@
 	)
 	(via
-		(at 165.735 97.79)
+		(at 165.735 98.425)
 		(size 0.7)
 		(drill 0.35)
@@
 	)
 	(segment
+		(start 154.958789 97.136211)
+		(end 157.558075 97.136211)
+		(width 0.2286)
+		(layer "B.Cu")
+		(net 13)
+	)
+	(segment
+		(start 165.753789 98.406211)
+		(end 165.735 98.425)
+		(width 0.2286)
+		(layer "B.Cu")
+		(net 13)
+	)
+	(segment
+		(start 165.51 98.2)
+		(end 165.735 98.425)
+		(width 0.2286)
+		(layer "B.Cu")
+		(net 13)
+	)
+	(segment
+		(start 172.103789 98.406211)
+		(end 165.753789 98.406211)
+		(width 0.2286)
+		(layer "B.Cu")
+		(net 13)
+	)
+	(segment
+		(start 158.621864 98.2)
+		(end 165.51 98.2)
+		(width 0.2286)
+		(layer "B.Cu")
+		(net 13)
+	)
+	(segment
 		(start 157.558075 97.136211)
+		(end 158.621864 98.2)
+		(width 0.2286)
+		(layer "B.Cu")
+		(net 13)
+	)
+	(segment
+		(start 153.035 99.06)
 		(end 154.958789 97.136211)
 		(width 0.2286)
@@
 	)
 	(segment
-		(start 166.351211 98.406211)
+		(start 176.53 93.98)
 		(end 172.103789 98.406211)
-		(width 0.2286)
-		(layer "B.Cu")
-		(net 13)
-	)
-	(segment
-		(start 165.325 98.2)
-		(end 158.621864 98.2)
-		(width 0.2286)
-		(layer "B.Cu")
-		(net 13)
-	)
-	(segment
-		(start 165.735 97.79)
-		(end 165.325 98.2)
-		(width 0.2286)
-		(layer "B.Cu")
-		(net 13)
-	)
-	(segment
-		(start 154.958789 97.136211)
-		(end 153.035 99.06)
-		(width 0.2286)
-		(layer "B.Cu")
-		(net 13)
-	)
-	(segment
-		(start 172.103789 98.406211)
-		(end 176.53 93.98)
-		(width 0.2286)
-		(layer "B.Cu")
-		(net 13)
-	)
-	(segment
-		(start 165.735 97.79)
-		(end 166.351211 98.406211)
-		(width 0.2286)
-		(layer "B.Cu")
-		(net 13)
-	)
-	(segment
-		(start 158.621864 98.2)
-		(end 157.558075 97.136211)
 		(width 0.2286)
 		(layer "B.Cu")
@@
 	)
 	(segment
-		(start 172.819489 98.980511)
-		(end 173.558467 98.241533)
-		(width 0.2286)
-		(layer "B.Cu")
-		(net 37)
-	)
-	(segment
 		(start 154.431022 100.203978)
 		(end 160.242898 100.203978)
@@
 	)
 	(segment
+		(start 173.123095 99.108438)
+		(end 161.338438 99.108438)
+		(width 0.2286)
+		(layer "B.Cu")
+		(net 37)
+	)
+	(segment
 		(start 177.616533 98.241533)
 		(end 178.435 99.06)
@@
 	)
 	(segment
-		(start 161.466365 98.980511)
-		(end 172.819489 98.980511)
+		(start 173.99 98.241533)
+		(end 173.123095 99.108438)
 		(width 0.2286)
 		(layer "B.Cu")
@@
 	)
 	(segment
-		(start 173.558467 98.241533)
+		(start 173.99 98.241533)
 		(end 177.616533 98.241533)
 		(width 0.2286)
@@
 	(segment
 		(start 160.242898 100.203978)
-		(end 161.466365 98.980511)
-		(width 0.2286)
-		(layer "B.Cu")
+		(end 161.338438 99.108438)
+		(width 0.2286)
+		(layer "B.Cu")

Commit message: Minor rev. d changes
Connections:
- U2 pad 22: unconnected-(U2-PB11-Pad22) -> BO0
- U3 pad 1: A15 -> A4
- U3 pad 2: B4 -> A6
- U3 pad 5: B5 -> A7
- U3 pad 6: B3 -> A5
Routing:
- net BO0: track 22.5 -> 46.4 mm, vias 2 -> 3
- net A7: track 6.29 -> 28.9 mm, vias 0 -> 2
- net A6: track 4.78 -> 25.8 mm, vias 0 -> 2
- net A5: track 3.95 -> 24.8 mm, vias 0 -> 2
- net A15: track 26.3 -> 6.94 mm, vias 2 -> 0
- net A4: track 4.94 -> 20.6 mm, vias 0 -> 2
- net B4: track 16.8 -> 4.25 mm, vias 1 -> 0
- net B5: track 16.2 -> 5.54 mm, vias 1 -> 0
- net C13: track 35.3 -> 43.7 mm
- net B3: track 34.6 -> 29.9 mm, vias 1 -> 0
- net RST: track 30.7 -> 32.6 mm
- net SWCLK: track 24.3 -> 25.2 mm
- net SWDIO: track 29.0 -> 29.6 mm
- net C15: track 19.2 -> 18.7 mm
- net GND: vias 21 -> 16
Other:
- board text added: "${TITLE}, rev. ${REVISION} STM32F103 Development Board © 2025 Lars Boegild Thomsen"
- board text removed: "${TITLE}, rev. ${REVISION} STM32 Development Board © 2025 Lars Boegild Thomsen"

Commit message: Hmmm
Routing:
- net +3V3: track 108.3 -> 57.8 mm, vias 2 -> 6
- net VBUS: track 13.2 -> 11.4 mm
- added copper zone on In1.Cu, net +3V3
- added copper zone on In2.Cu, net GND
Other:
- copper layers 2 -> 4
Changed lines of the file:
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@@
 	(generator_version "9.0")
 	(general
-		(thickness 1.6)
+		(thickness 1.2)
 		(legacy_teardrops no)
 	)
@@
 	(layers
 		(0 "F.Cu" signal)
+		(4 "In1.Cu" signal)
+		(6 "In2.Cu" signal)
 		(2 "B.Cu" signal)
 		(9 "F.Adhes" user "F.Adhesive")
@@
 			)
 			(layer "dielectric 1"
+				(type "prepreg")
+				(thickness 0.1)
+				(material "FR4")
+				(epsilon_r 4.5)
+				(loss_tangent 0.02)
+			)
+			(layer "In1.Cu"
+				(type "copper")
+				(thickness 0.035)
+			)
+			(layer "dielectric 2"
 				(type "core")
-				(thickness 1.51)
+				(thickness 0.84)
+				(material "FR4")
+				(epsilon_r 4.5)
+				(loss_tangent 0.02)
+			)
+			(layer "In2.Cu"
+				(type "copper")
+				(thickness 0.035)
+			)
+			(layer "dielectric 3"
+				(type "prepreg")
+				(thickness 0.1)
 				(material "FR4")
 				(epsilon_r 4.5)
@@
 	)
 	(segment
-		(start 194.2927 105.4273)
-		(end 194.2927 104.51914)
-		(width 0.2286)
+		(start 197.817593 103.562901)
+		(end 198.28 103.100494)
+		(width 0.381)
 		(layer "F.Cu")
 		(net 2)
 	)
 	(segment
-		(start 197.817593 103.562901)
-		(end 198.28 103.100494)
+		(start 195.98 104.05)
+		(end 194.84 104.05)
 		(width 0.381)
 		(layer "F.Cu")
@@
 	)
 	(segment
-		(start 195.98 104.05)
-		(end 193.33 104.05)
+		(start 194.55 103.76)
+		(end 194.84 104.05)
 		(width 0.381)
 		(layer "F.Cu")
@@
 	)
 	(segment
-		(start 197.259321 103.562901)
-		(end 197.817593 103.562901)
+		(start 193.04 103.76)
+		(end 194.55 103.76)
 		(width 0.381)
 		(layer "F.Cu")
@@
 	)
 	(segment
-		(start 196.772222 104.05)
-		(end 197.259321 103.562901)
+		(start 197.259321 103.562901)
+		(end 197.817593 103.562901)
 		(width 0.381)
 		(layer "F.Cu")
@@
 	)
 	(segment
-		(start 193.675 106.045)
-		(end 194.2927 105.4273)
-		(width 0.2286)
+		(start 196.772222 104.05)
+		(end 197.259321 103.562901)
+		(width 0.381)
 		(layer "F.Cu")
 		(net 2)
@@
 		(net 2)
 	)
-	(segment
-		(start 193.33 104.05)
-		(end 193.04 103.76)
-		(width 0.381)
-		(layer "F.Cu")
-		(net 2)
-	)
-	(segment
-		(start 194.2927 104.51914)
-		(end 194.28176 104.5082)
-		(width 0.2286)
-		(layer "F.Cu")
-		(net 2)
-	)
 	(via
 		(at 192.405 104.775)
@@
 	)
 	(segment
+		(start 176.143883 104.388883)
+		(end 175.105551 105.427215)
+		(width 0.3048)
+		(layer "F.Cu")
+		(net 3)
+	)
+	(segment
 		(start 172.085 101.6)
 		(end 172.085 102.406664)
@@
 	)
 	(segment
-		(start 172.085 102.406664)
-		(end 172.277124 102.598788)
-		(width 0.3048)
+		(start 159.385 100.625)
+		(end 159.385 99.695)
+		(width 0.381)
 		(layer "F.Cu")
 		(net 3)
 	)
 	(segment
-		(start 177.165 97.710912)
-		(end 178.163788 96.712124)
+		(start 172.085 102.406664)
+		(end 172.277124 102.598788)
 		(width 0.3048)
 		(layer "F.Cu")
@@
 	)
 	(segment
-		(start 154.227901 102.222099)
-		(end 154.227901 100.407099)
-		(width 0.381)
-		(layer "F.Cu")
-		(net 3)
-	)
-	(segment
 		(start 159.725 100.965)
 		(end 159.385 100.625)
@@
 	)
 	(segment
-		(start 154.227901 100.407099)
-		(end 154.227901 94.537901)
-		(width 0.381)
-		(layer "F.Cu")
-		(net 3)
-	)
-	(segment
 		(start 189.5 101.6)
 		(end 187.325 101.6)
@@
 	)
 	(segment
-		(start 153.035 103.415)
-		(end 154.227901 102.222099)
-		(width 0.381)
-		(layer "F.Cu")
-		(net 3)
-	)
-	(segment
 		(start 178.990912 95.885)
 		(end 178.163788 96.712124)
@@
 	)
 	(segment
-		(start 177.165 103.367766)
-		(end 175.105551 105.427215)
-		(width 0.3048)
-		(layer "F.Cu")
-		(net 3)
-	)
-	(segment
-		(start 177.165 101.6)
-		(end 177.165 97.710912)
-		(width 0.3048)
-		(layer "F.Cu")
-		(net 3)
-	)
-	(segment
 		(start 193.165 98.425)
 		(end 190.0175 98.425)
@@
 	)
 	(segment
-		(start 172.105 101.58)
-		(end 177.145 101.58)
-		(width 0.3048)
-		(layer "F.Cu")
-		(net 3)
-	)
-	(segment
 		(start 172.085 101.6)
 		(end 172.085 100.793336)
@@
 	)
 	(segment
-		(start 177.165 101.6)
-		(end 177.165 103.367766)
-		(width 0.3048)
-		(layer "F.Cu")
-		(net 3)
-	)
-	(segment
 		(start 187.01 103.14)
 		(end 187.01 101.915)
@@
 	)
 	(segment
-		(start 154.227901 100.407099)
-		(end 159.167099 100.407099)
-		(width 0.2286)
+		(start 179.07 95.885)
+		(end 178.990912 95.885)
+		(width 0.3048)
 		(layer "F.Cu")
 		(net 3)
@@
 	(segment
 		(start 179.855 95.885)
-		(end 178.990912 95.885)
+		(end 179.07 95.885)
 		(width 0.3048)
 		(layer "F.Cu")
@@
 	)
 	(segment
-		(start 182.052876 102.598788)
-		(end 181.054088 101.6)
-		(width 0.3048)
-		(layer "F.Cu")
-		(net 3)
-	)
-	(segment
-		(start 181.054088 101.6)
-		(end 177.165 101.6)
-		(width 0.3048)
-		(layer "F.Cu")
-		(net 3)
-	)
-	(segment
 		(start 172.085 100.793336)
 		(end 172.277124 100.601212)
@@
 	)
 	(segment
-		(start 153.185 106.68)
-		(end 153.185 104.29)
-		(width 0.381)
+		(start 184.15 103.365)
+		(end 182.819088 103.365)
+		(width 0.3048)
 		(layer "F.Cu")
 		(net 3)
@@
 	(segment
 		(start 185.42 103.365)
-		(end 182.819088 103.365)
+		(end 184.15 103.365)
 		(width 0.3048)
 		(layer "F.Cu")
@@
 	)
 	(via
+		(at 179.07 95.885)
+		(size 0.7)
+		(drill 0.35)
+		(layers "F.Cu" "B.Cu")
+		(net 3)
+	)
+	(via
 		(at 172.085 101.6)
 		(size 0.7)
@@
 	)
 	(via
+		(at 176.143883 104.388883)
+		(size 0.7)
+		(drill 0.35)
+		(layers "F.Cu" "B.Cu")
+		(net 3)
+	)
+	(via
 		(at 187.325 101.6)
 		(size 0.7)
@@
 		(net 3)
 	)
+	(via
+		(at 159.385 99.695)
+		(size 0.7)
+		(drill 0.35)
+		(layers "F.Cu" "B.Cu")
+		(net 3)
+	)
+	(via
+		(at 184.15 103.365)
+		(size 0.7)
+		(drill 0.35)
+		(layers "F.Cu" "B.Cu")
+		(net 3)
+	)
 	(segment
 		(start 154.305 105.41)
@@
 	)
 	(segment
-		(start 194.95 101.68)
-		(end 187.405 101.68)
-		(width 0.381)
-		(layer "B.Cu")
-		(net 3)
-	)
-	(segment
-		(start 196.85 109.22)
-		(end 195.34 107.71)
-		(width 0.381)
-		(layer "B.Cu")
-		(net 3)
-	)
-	(segment
-		(start 195.34 102.07)
-		(end 194.95 101.68)
-		(width 0.381)
-		(layer "B.Cu")
-		(net 3)
-	)
-	(segment
 		(start 168.609106 101.6)
 		(end 164.799106 105.41)
@@
 	)
 	(segment
-		(start 195.34 107.71)
-		(end 195.34 102.07)
-		(width 0.381)
-		(layer "B.Cu")
-		(net 3)
-	)
-	(segment
 		(start 187.405 101.68)
 		(end 187.325 101.6)
@@
 		(net 1)
 		(net_name "GND")
-		(layers "F.Cu" "B.Cu")
+		(layers "F.Cu" "B.Cu" "In2.Cu")
 		(hatch edge 0.508)
 		(connect_pads
@@
 			)
 		)
+	)
+	(zone
+		(net 3)
+		(net_name "+3V3")
+		(layer "In1.Cu")
+		(hatch edge 0.508)
+		(priority 3)
+		(connect_pads
+			(clearance 0.1524)
+		)
+		(min_thickness 0.1524)
+		(filled_areas_thickness no)
+		(fill yes
+			(thermal_gap 0.1524)
+			(thermal_bridge_width 0.3048)
+		)
+		(polygon
+			(pts
+				(xy 150.495 86.995) (xy 205.105 86.995) (xy 205.105 114.3) (xy 150.495 114.3)
+			)
+		)

Commit message: More fine tuning of PCB
Parts:
- D2: value GRE -> WHI
- moved C4 2.62 mm to (184.2, 104.1), turned to -90 degrees
- moved C6 1.42 mm to (171.4, 106.7)
Routing:
- net BO0: track 46.4 -> 31.3 mm, vias 3 -> 2
- net +3V3: track 57.8 -> 51.4 mm, vias 6 -> 10
- net C13: track 43.7 -> 38.2 mm, vias 2 -> 3
- net RST: track 32.6 -> 29.5 mm, vias 0 -> 2
- net GND: vias 16 -> 17

Commit message: Tweaks
Parts:
- added C4: 100nF, Capacitor_SMD:C_0402_1005Metric, F.Cu at (153.5, 96.5)
- added C9: 100nF, Capacitor_SMD:C_0402_1005Metric, F.Cu at (162.1, 103.6)
- renumbered C8 to C10, C9 to C11, C4 to C5, C5 to C6, C6 to C7, C7 to C8, R5 to R2, R2 to R3, R3 to R4, R4 to R5, R8 to R6, R6 to R7, R9 to R8, R7 to R9, U3 to U2, U2 to U3
Routing:
- net +3V3: track 51.4 -> 30.1 mm, vias 10 -> 11
- net BO0: track 31.3 -> 34.2 mm
- net C14: track 20.9 -> 20.2 mm
- net C15: track 18.6 -> 17.8 mm
- net GND: vias 17 -> 23
